Commit message: working model in gazebo

File: hovermower_description/urdf/hovermower.urdf (robot description, URDF)
Before this commit: robot HoverMower, 10 links, 9 joints
Links:
- link base_footprint: geometry visual box size=0.010 0.010 0.010

Commit message: gazebo fixes

File: hovermower_description/urdf/hovermower.urdf (robot description, URDF)
Before this commit: robot HoverMower, 10 links, 9 joints
Links:
- added link caster_wheel; collision sphere radius=${caster_wheel_radius}; visual sphere radius=${caster_wheel_radius}
Joints:
- added joint caster_wheel_joint: type fixed, parent base_link, child caster_wheel, origin xyz=${caster_wheel_joint_offset_x} ${caster_wheel_joint_offset_y} ${caster_wheel_joint_offset_z}
